File: KiCad/211027.sch (KiCad schematic (older format))
At the start: 1 part

Commit message: update schematics and libraries
Parts:
- gave numbers to parts that had none: 1
Changed lines of the file:
@@
 $EndDescr
 $Comp
-L Device:R R?
+L Device:R R1
 U 1 1 6178C86A
 P 5800 3150
-F 0 "R?" H 5870 3196 50  0000 L CNN
+F 0 "R1" H 5870 3196 50  0000 L CNN
 F 1 "R" H 5870 3105 50  0000 L CNN
 F 2 "" V 5730 3150 50  0001 C CNN
