File: KiCad/eq_NPN.sch (KiCad schematic (older format))
At the start: 7 parts

Commit message: resume + exercices
Other:
- note added: "charge"
- note added: "transistor"
Changed lines of the file:
@@
 	1    0    0    -1
 $EndComp
+Wire Notes Line
+	1800 2350 4000 2350
+Wire Notes Line
+	4000 2350 4000 3100
+Wire Notes Line
+	4000 3100 1800 3100
+Wire Notes Line
+	1800 3100 1800 2350
+Text Notes 2650 2450 0    50   ~ 0
+transistor
+Text Notes 4050 2450 0    50   ~ 0
+charge
 $EndSCHEMATC
