File: KiCad/211026.sch (KiCad schematic (older format))
At the start: 0 parts

Commit message: 220122
Other:
- note added: "validé"
- note added: "validé\n"
Changed lines of the file:
@@
 $Descr A4 11693 8268
 encoding utf-8
-Sheet 2 12
+Sheet 2 16
 Title ""
 Date ""
@@
 Text Notes 3000 1350 0    50   ~ 0
 Différentiel avec\nalimentation unipolaire\n
+Text Notes 3300 1850 0    50   ~ 0
+validé\n
+Text Notes 1050 1850 0    50   ~ 0
+validé
+Text Notes 2350 1850 0    50   ~ 0
+validé
 $EndSCHEMATC
