File: KiCad/220122.sch (KiCad schematic (older format))
At the start: 0 parts

Commit message: exercices + resume
Changed lines of the file:
@@
 $Descr A4 11693 8268
 encoding utf-8
-Sheet 14 16
+Sheet 14 18
 Title ""
 Date ""
@@
 Text Notes 1950 1750 0    50   ~ 0
 validé
+$Sheet
+S 2500 650  750  900
+U 61ED736D
+F0 "220122_03" 50
+F1 "220122_03.sch" 50
+$EndSheet
+$Sheet
+S 3300 650  650  900
+U 61ED926F
+F0 "220122_04" 50
+F1 "220122_04.sch" 50
+$EndSheet
 $EndSCHEMATC
