File: KiCad/220122_02.sch (KiCad schematic (older format))
At the start: 3 parts

Commit message: exercices + resume
Connections:
- net Uout: now reaches R?.1, U?.3
Changed lines of the file:
@@
 $Descr A4 11693 8268
 encoding utf-8
-Sheet 16 16
+Sheet 16 18
 Title ""
 Date ""
@@
 Wire Wire Line
 	2350 1600 2300 1600
+Text GLabel 2350 1600 2    50   Input ~ 0
+Uout
 $EndSCHEMATC
