File: KiCad/resume.sch (KiCad schematic (older format))
At the start: 0 parts

Commit message: 220122
Changed lines of the file:
@@
 $Descr A4 11693 8268
 encoding utf-8
-Sheet 1 12
+Sheet 1 16
 Title ""
 Date ""
@@
 F1 "220108.sch" 50
 $EndSheet
+$Sheet
+S 3550 750  700  550
+U 61EC4A71
+F0 "220122" 50
+F1 "220122.sch" 50
+$EndSheet
 $EndSCHEMATC
